File: Hardware/Cynara Viride.sch (EAGLE design)
At the start: 192 parts, among them Q1 TXC-7B, Q2 TXC-7WNEO, SW1 430181038816, SW2 , T1 PDTC143, T2 PDTC143, T3 PDTC143, T4 PDTC143, T5 PDTC143, U1 TM4C129EN, U2 MCP1826S 3V3, U3 LM4132 3V3, U4 XC6SLX9-3TQG, U5 M25P16-SO8, U6 MCP1826S 1V2, X1 EDGE 50p, X11 SOCK2X17, X12 SOCK2X17, X13 SOCK2X17, X2 EDGE 50p, X23 debug xilinx, X24 debug 10p, X3 EDGE 50p, X4 EDGE 50p, X5 MicroMatch 24, X6 , X7 SOCK2X17, X8 RJ45-LAN-10/100

Commit message: Changed microcontroller symbol to one a functional and power part. Renamed Petal signals. Shield for Ethernet and USB is a polygon now.
Parts:
- added TP1, TP2, TP3, TP4, TP5: (no value), Cynara-Misc:TESTPAD-SMD
Connections:
- net FPGA_III_A renamed FPGA_III_1
- net FPGA_III_B renamed FPGA_III_2
- net FPGA_III_C renamed FPGA_III_3
- net FPGA_III_D renamed FPGA_III_4
- net FPGA_III_E renamed FPGA_III_5
- net FPGA_III_F renamed FPGA_III_6
- net FPGA_III_G renamed FPGA_III_7
- net FPGA_III_H renamed FPGA_III_8
- net FPGA_III_I renamed FPGA_III_9
- net FPGA_III_J renamed FPGA_III_10
- net FPGA_III_K renamed FPGA_III_11
- net FPGA_III_L renamed FPGA_III_12
- net FPGA_III_M renamed FPGA_III_13
- net FPGA_III_N renamed FPGA_III_14
- net FPGA_III_O renamed FPGA_III_15
- net FPGA_III_P renamed FPGA_III_16
- net FPGA_IV_A renamed FPGA_IV_1
- net FPGA_IV_B renamed FPGA_IV_2
- net FPGA_IV_C renamed FPGA_IV_3
- net FPGA_IV_D renamed FPGA_IV_4
- net FPGA_IV_E renamed FPGA_IV_5
- net FPGA_IV_F renamed FPGA_IV_6
- net FPGA_IV_G renamed FPGA_IV_7
- net FPGA_IV_H renamed FPGA_IV_8
- net FPGA_IV_I renamed FPGA_IV_9
- net FPGA_IV_J renamed FPGA_IV_10
- net FPGA_IV_K renamed FPGA_IV_11
- net FPGA_IV_L renamed FPGA_IV_12
- net FPGA_IV_M renamed FPGA_IV_13
- net FPGA_IV_N renamed FPGA_IV_14
- net FPGA_IV_O renamed FPGA_IV_15
- net FPGA_IV_P renamed FPGA_IV_16
- net PETAL_III_A renamed PETAL_III_1
- net PETAL_III_B renamed PETAL_III_2
- net PETAL_III_C renamed PETAL_III_3
- net PETAL_III_D renamed PETAL_III_4
- net PETAL_III_E renamed PETAL_III_5
- net PETAL_III_F renamed PETAL_III_6
- net PETAL_III_G renamed PETAL_III_7
- net PETAL_III_H renamed PETAL_III_8
- net PETAL_III_I renamed PETAL_III_9
- net PETAL_III_J renamed PETAL_III_10
- net PETAL_III_K renamed PETAL_III_11
- net PETAL_III_L renamed PETAL_III_12
- net PETAL_III_M renamed PETAL_III_13
- net PETAL_III_N renamed PETAL_III_14
- net PETAL_III_O renamed PETAL_III_15
- net PETAL_III_P renamed PETAL_III_16
- net PETAL_III_Q renamed PETAL_III_17
- net PETAL_III_R renamed PETAL_III_18
- net PETAL_III_S renamed PETAL_III_19
- net PETAL_III_T renamed PETAL_III_20
- net PETAL_III_U renamed PETAL_III_21
- net PETAL_III_V renamed PETAL_III_22
- net PETAL_III_W renamed PETAL_III_23
- net PETAL_III_X renamed PETAL_III_24
- net PETAL_III_Y renamed PETAL_III_25
- net PETAL_III_Z renamed PETAL_III_26
- net PETAL_II_A renamed PETAL_II_1
- net PETAL_II_B renamed PETAL_II_2
- net PETAL_II_C renamed PETAL_II_3
- net PETAL_II_D renamed PETAL_II_4
- net PETAL_II_E renamed PETAL_II_5
- net PETAL_II_F renamed PETAL_II_6
- net PETAL_II_G renamed PETAL_II_7
- net PETAL_II_H renamed PETAL_II_8
- net PETAL_II_I renamed PETAL_II_9
- net PETAL_II_J renamed PETAL_II_10
- net PETAL_II_K renamed PETAL_II_11
- net PETAL_II_L renamed PETAL_II_12
- net PETAL_II_M renamed PETAL_II_13
- net PETAL_II_N renamed PETAL_II_14
- net PETAL_II_O renamed PETAL_II_15
- net PETAL_II_P renamed PETAL_II_16
- net PETAL_II_Q renamed PETAL_II_17
- net PETAL_II_R renamed PETAL_II_18
- net PETAL_II_S renamed PETAL_II_19
- net PETAL_II_T renamed PETAL_II_20
- net PETAL_II_U renamed PETAL_II_21
- net PETAL_II_V renamed PETAL_II_22
- net PETAL_II_W renamed PETAL_II_23
- net PETAL_II_X renamed PETAL_II_24
- net PETAL_II_Y renamed PETAL_II_25
- net PETAL_II_Z renamed PETAL_II_26
- net PETAL_IV_A renamed PETAL_IV_1
- net PETAL_IV_B renamed PETAL_IV_2
- net PETAL_IV_C renamed PETAL_IV_3
- net PETAL_IV_D renamed PETAL_IV_4
- net PETAL_IV_E renamed PETAL_IV_5
- net PETAL_IV_F renamed PETAL_IV_6
- net PETAL_IV_G renamed PETAL_IV_7
- net PETAL_IV_H renamed PETAL_IV_8
- net PETAL_IV_I renamed PETAL_IV_9
- net PETAL_IV_J renamed PETAL_IV_10
- net PETAL_IV_K renamed PETAL_IV_11
- net PETAL_IV_L renamed PETAL_IV_12
- net PETAL_IV_M renamed PETAL_IV_13
- net PETAL_IV_N renamed PETAL_IV_14
- net PETAL_IV_O renamed PETAL_IV_15
- net PETAL_IV_P renamed PETAL_IV_16
- net PETAL_IV_Q renamed PETAL_IV_17
- net PETAL_IV_R renamed PETAL_IV_18
- net PETAL_IV_S renamed PETAL_IV_19
- net PETAL_IV_T renamed PETAL_IV_20
- net PETAL_IV_U renamed PETAL_IV_21
- net PETAL_IV_V renamed PETAL_IV_22
- net PETAL_IV_W renamed PETAL_IV_23
- net PETAL_IV_X renamed PETAL_IV_24
- net PETAL_IV_Y renamed PETAL_IV_25
- net PETAL_IV_Z renamed PETAL_IV_26
- net PETAL_I_A renamed PETAL_I_1
- net PETAL_I_B renamed PETAL_I_2
- net PETAL_I_C renamed PETAL_I_3
- net PETAL_I_D renamed PETAL_I_4
- net PETAL_I_E renamed PETAL_I_5
- net PETAL_I_F renamed PETAL_I_6
- net PETAL_I_G renamed PETAL_I_7
- net PETAL_I_H renamed PETAL_I_8
- net PETAL_I_I renamed PETAL_I_9
- net PETAL_I_J renamed PETAL_I_10
- net PETAL_I_K renamed PETAL_I_11
- net PETAL_I_L renamed PETAL_I_12
- net PETAL_I_M renamed PETAL_I_13
- net PETAL_I_N renamed PETAL_I_14
- net PETAL_I_O renamed PETAL_I_15
- net PETAL_I_P renamed PETAL_I_16
- net PETAL_I_Q renamed PETAL_I_17
- net PETAL_I_R renamed PETAL_I_18
- net PETAL_I_S renamed PETAL_I_19
- net PETAL_I_T renamed PETAL_I_20
- net PETAL_I_U renamed PETAL_I_21
- net PETAL_I_V renamed PETAL_I_22
- net PETAL_I_W renamed PETAL_I_23
- net PETAL_I_X renamed PETAL_I_24
- net PETAL_I_Y renamed PETAL_I_25
- net PETAL_I_Z renamed PETAL_I_26
- removed net FREE: U1J.PJ0
- removed net MCU_II_A: RA17.1B, U1B.PB1
- removed net MCU_II_B: RA17.2B, U1B.PB0
- removed net MCU_II_C: RA17.3B, U1N.PN0
- removed net MCU_II_D: RA17.4B, U1N.PN1
- removed net MCU_II_E: RA18.1B, U1N.PN2
- removed net MCU_II_F: RA18.2B, U1N.PN3
- removed net MCU_II_G: RA18.3B, U1N.PN4
- removed net MCU_II_H: RA18.4B, U1N.PN5
- removed net MCU_II_I: RA19.1B, U1M.PM6
- removed net MCU_II_J: RA19.2B, U1M.PM7
- removed net MCU_II_K: RA20.1A, U1B.PB5
- removed net MCU_II_L: RA20.2A, U1B.PB4
- removed net MCU_II_M: RA20.3A, U1E.PE4
- removed net MCU_II_N: RA20.4A, U1E.PE5
- removed net MCU_II_O: RA21.1A, U1D.PD4
- removed net MCU_II_P: RA21.2A, U1D.PD5
- removed net MCU_I_A: RA10.1B, U1A.PA1
- removed net MCU_I_B: RA10.2B, U1A.PA0
- removed net MCU_I_C: RA10.3B, U1H.PH0
- removed net MCU_I_D: RA10.4B, U1H.PH1
- removed net MCU_I_E: RA11.1B, U1E.PE0
- removed net MCU_I_F: RA11.2B, U1E.PE1
- removed net MCU_I_G: RA11.3B, U1E.PE2
- removed net MCU_I_H: RA11.4B, U1E.PE3
- removed net MCU_I_I: RA12.1B, U1M.PM4
- removed net MCU_I_J: RA12.2B, U1M.PM5
- removed net MCU_I_K: RA13.1B, U1D.PD3
- removed net MCU_I_L: RA13.2B, U1D.PD2
- removed net MCU_I_M: RA13.3B, U1D.PD1
- removed net MCU_I_N: RA13.4B, U1D.PD0
- removed net MCU_I_O: RA14.1B, U1D.PD7
- removed net MCU_I_P: RA14.2B, U1D.PD6
- removed net N$10: C50.1, Q1.XTALB, U1O.OSC1
- removed net N$7: R12.2, U1O.OSC0
- removed net N$79: C60.1, L2.E, U1S.VDDA
- removed net N$84: L1.E, U1S.GNDA
- removed net OLED_CS: U4D.IO_L83N_VREF
- removed net OLED_DC: U4D.IO_L52N
- removed net OLED_MOSI: U4D.IO_L51N
- removed net OLED_RST: U4D.IO_L83P
- removed net OLED_SCLK: U4D.IO_L52P
- removed net VDCC: C45.1, C46.1, C47.1, C48.1, U1S.VDDC@115, U1S.VDDC@87
- new net GNDA: L1.E, U1-POWER.GNDA
- new net MCU_II_1: RA17.1B, U1-FUNCTIONAL.PB1
- new net MCU_II_10: RA19.2B, U1-FUNCTIONAL.PM7
- new net MCU_II_11: RA20.1A, U1-FUNCTIONAL.PB5
- new net MCU_II_12: RA20.2A, U1-FUNCTIONAL.PB4
- new net MCU_II_13: RA20.3A, U1-FUNCTIONAL.PE4
- new net MCU_II_14: RA20.4A, U1-FUNCTIONAL.PE5
- new net MCU_II_15: RA21.1A, U1-FUNCTIONAL.PD4
- new net MCU_II_16: RA21.2A, U1-FUNCTIONAL.PD5
- new net MCU_II_2: RA17.2B, U1-FUNCTIONAL.PB0
- new net MCU_II_3: RA17.3B, U1-FUNCTIONAL.PN0
- new net MCU_II_4: RA17.4B, U1-FUNCTIONAL.PN1
- new net MCU_II_5: RA18.1B, U1-FUNCTIONAL.PN2
- new net MCU_II_6: RA18.2B, U1-FUNCTIONAL.PN3
- new net MCU_II_7: RA18.3B, U1-FUNCTIONAL.PN4
- new net MCU_II_8: RA18.4B, U1-FUNCTIONAL.PN5
- new net MCU_II_9: RA19.1B, U1-FUNCTIONAL.PM6
- new net MCU_I_1: RA10.1B, U1-FUNCTIONAL.PA1
- new net MCU_I_10: RA12.2B, U1-FUNCTIONAL.PM5
- new net MCU_I_11: RA13.1B, U1-FUNCTIONAL.PD3
- new net MCU_I_12: RA13.2B, U1-FUNCTIONAL.PD2
- new net MCU_I_13: RA13.3B, U1-FUNCTIONAL.PD1
- new net MCU_I_14: RA13.4B, U1-FUNCTIONAL.PD0
- new net MCU_I_15: RA14.1B, U1-FUNCTIONAL.PD7
- new net MCU_I_16: RA14.2B, U1-FUNCTIONAL.PD6
- new net MCU_I_2: RA10.2B, U1-FUNCTIONAL.PA0
- new net MCU_I_3: RA10.3B, U1-FUNCTIONAL.PH0
- new net MCU_I_4: RA10.4B, U1-FUNCTIONAL.PH1
- new net MCU_I_5: RA11.1B, U1-FUNCTIONAL.PE0
- new net MCU_I_6: RA11.2B, U1-FUNCTIONAL.PE1
- new net MCU_I_7: RA11.3B, U1-FUNCTIONAL.PE2
- new net MCU_I_8: RA11.4B, U1-FUNCTIONAL.PE3
- new net MCU_I_9: RA12.1B, U1-FUNCTIONAL.PM4
- new net OSC0: R12.2, U1-FUNCTIONAL.OSC0
- new net OSC1: C50.1, Q1.XTALB, U1-FUNCTIONAL.OSC1
- new net VDDA: C60.1, L2.E, U1-POWER.VDDA
- new net VDDC: C45.1, C46.1, C47.1, C48.1, U1-POWER.VDDC@115, U1-POWER.VDDC@87
- net !HIB: now also U1-FUNCTIONAL.!HIB; no longer U1O.!HIB
- net !RST: now also U1-FUNCTIONAL.!RST; no longer U1O.!RST
- net !WAKE: now also U1-FUNCTIONAL.!WAKE; no longer U1O.!WAKE
- net +1.2V: now also TP3.1
- net +3.3V: now also TP2.1, U1-POWER.VBAT, U1-POWER.VDD@101, U1-POWER.VDD@113, U1-POWER.VDD@122, U1-POWER.VDD@16, U1-POWER.VDD@26, U1-POWER.VDD@28, U1-POWER.VDD@39, U1-POWER.VDD@47, U1-POWER.VDD@51, U1-POWER.VDD@52, U1-POWER.VDD@69, U1-POWER.VDD@7, U1-POWER.VDD@79, U1-POWER.VDD@90; no longer U1S.VBAT, U1S.VDD@101, U1S.VDD@113, U1S.VDD@122, U1S.VDD@16, U1S.VDD@26, U1S.VDD@28, U1S.VDD@39, U1S.VDD@47, U1S.VDD@51, U1S.VDD@52, U1S.VDD@69, U1S.VDD@7, U1S.VDD@79, U1S.VDD@90
- net +5V: now also TP1.1
- net DONE: now also U1-FUNCTIONAL.PH3; no longer U1H.PH3
- net EPI0S0: now also U1-FUNCTIONAL.PK0; no longer U1K.PK0
- net EPI0S1: now also U1-FUNCTIONAL.PK1; no longer U1K.PK1
- net EPI0S10: now also U1-FUNCTIONAL.PG1; no longer U1G.PG1
- net EPI0S11: now also U1-FUNCTIONAL.PG0; no longer U1G.PG0
- net EPI0S12: now also U1-FUNCTIONAL.PM3; no longer U1M.PM3
- net EPI0S13: now also U1-FUNCTIONAL.PM2; no longer U1M.PM2
- net EPI0S14: now also U1-FUNCTIONAL.PM1; no longer U1M.PM1
- net EPI0S15: now also U1-FUNCTIONAL.PM0; no longer U1M.PM0
- net EPI0S16: now also U1-FUNCTIONAL.PL0; no longer U1L.PL0
- net EPI0S17: now also U1-FUNCTIONAL.PL1; no longer U1L.PL1
- net EPI0S18: now also U1-FUNCTIONAL.PL2; no longer U1L.PL2
- net EPI0S19: now also U1-FUNCTIONAL.PL3; no longer U1L.PL3
- net EPI0S2: now also U1-FUNCTIONAL.PK2; no longer U1K.PK2
- net EPI0S20: now also U1-FUNCTIONAL.PQ0; no longer U1Q.PQ0
- net EPI0S21: now also U1-FUNCTIONAL.PQ1; no longer U1Q.PQ1
- net EPI0S22: now also U1-FUNCTIONAL.PQ2; no longer U1Q.PQ2
- net EPI0S23: now also U1-FUNCTIONAL.PQ3; no longer U1Q.PQ3
- net EPI0S24: now also U1-FUNCTIONAL.PK7; no longer U1K.PK7
- net EPI0S25: now also U1-FUNCTIONAL.PK6; no longer U1K.PK6
- net EPI0S26: now also U1-FUNCTIONAL.PL4; no longer U1L.PL4
- net EPI0S27: now also U1-FUNCTIONAL.PB2; no longer U1B.PB2
- net EPI0S28: now also U1-FUNCTIONAL.PB3; no longer U1B.PB3
- net EPI0S29: now also U1-FUNCTIONAL.PP2; no longer U1P.PP2
- net EPI0S3: now also U1-FUNCTIONAL.PK3; no longer U1K.PK3
- net EPI0S30: now also U1-FUNCTIONAL.PP3; no longer U1P.PP3
- net EPI0S31: now also U1-FUNCTIONAL.PK5; no longer U1K.PK5
- net EPI0S4: now also U1-FUNCTIONAL.PC7; no longer U1C.PC7
- net EPI0S5: now also U1-FUNCTIONAL.PC6; no longer U1C.PC6
- net EPI0S6: now also U1-FUNCTIONAL.PC5; no longer U1C.PC5
- net EPI0S7: now also U1-FUNCTIONAL.PC4; no longer U1C.PC4
- net EPI0S8: now also U1-FUNCTIONAL.PA6; no longer U1A.PA6
- net EPI0S9: now also U1-FUNCTIONAL.PA7; no longer U1A.PA7
- net ETH_PAIR0_N: now also U1-FUNCTIONAL.EN0TXON; no longer U1I.EN0TXON
- net ETH_PAIR0_P: now also U1-FUNCTIONAL.EN0TXOP; no longer U1I.EN0TXOP
- net ETH_PAIR1_N: now also U1-FUNCTIONAL.EN0RXIN; no longer U1I.EN0RXIN
- net ETH_PAIR1_P: now also U1-FUNCTIONAL.EN0RXIP; no longer U1I.EN0RXIP
- net GND: now also TP4.1, TP5.1, U1-POWER.GND@114, U1-POWER.GND@17, U1-POWER.GND@48, U1-POWER.GND@55, U1-POWER.GND@58, U1-POWER.GND@80, U2.GND, U6.GND, X8-RJ45-LAN.SH; no longer U1S.GND@114, U1S.GND@17, U1S.GND@48, U1S.GND@55, U1S.GND@58, U1S.GND@80, U2.GND1, U6.GND1
- net INIT: now also U1-FUNCTIONAL.PL5; no longer U1L.PL5
- net MCU_TCK: now also U1-FUNCTIONAL.PC0/TCK/SWCLK; no longer U1C.PC0/TCK/SWCLK
- net MCU_TDI: now also U1-FUNCTIONAL.PC2/TDI; no longer U1C.PC2/TDI
- net MCU_TDO: now also U1-FUNCTIONAL.PC3/TDO/SWO; no longer U1C.PC3/TDO/SWO
- net MCU_TMS: now also U1-FUNCTIONAL.PC1/TMS/SWDIO; no longer U1C.PC1/TMS/SWDIO
- net PF0_ETH: now also U1-FUNCTIONAL.PF0; no longer U1F.PF0
- net PF1_LEDR: now also U1-FUNCTIONAL.PF1; no longer U1F.PF1
- net PF2_LEDB: now also U1-FUNCTIONAL.PF2; no longer U1F.PF2
- net PF3_LEDG: now also U1-FUNCTIONAL.PF3; no longer U1F.PF3
- net PF4_ETH: now also U1-FUNCTIONAL.PF4; no longer U1F.PF4
- net PJ1_FLASHWP: now also U1-FUNCTIONAL.PJ1; no longer U1J.PJ1
- net PROGRAM: now also U1-FUNCTIONAL.PH2; no longer U1H.PH2
- net RBIAS: now also U1-FUNCTIONAL.RBIAS; no longer U1I.RBIAS
- net RUPT0: now also U1-FUNCTIONAL.PP0; no longer U1P.PP0
- net RUPT1: now also U1-FUNCTIONAL.PP1; no longer U1P.PP1
- net RUPT2: now also U1-FUNCTIONAL.PP4; no longer U1P.PP4
- net RUPT3: now also U1-FUNCTIONAL.PP5; no longer U1P.PP5
- net SSI0CLK: now also U1-FUNCTIONAL.PA2; no longer U1A.PA2
- net SSI0D0: now also U1-FUNCTIONAL.PA4; no longer U1A.PA4
- net SSI0D1: now also U1-FUNCTIONAL.PA5; no longer U1A.PA5
- net SSI0FSS: now also U1-FUNCTIONAL.PA3; no longer U1A.PA3
- net USB0D_N: now also U1-FUNCTIONAL.PL7; no longer U1L.PL7
- net USB0D_P: now also U1-FUNCTIONAL.PL6; no longer U1L.PL6
- net USB_DETECT: now also U1-FUNCTIONAL.PK4; no longer U1K.PK4
- net VREFA+: now also U1-POWER.VREFA+; no longer U1S.VREFA+
Other:
- note removed: "calculate xtal caps"
- note removed: "calculate xtal res"
- note removed: "find rtc xtal"
